Commit message: commented new thruster positions for future use

File: simulator/descriptions/urab_sub_description/urdf/urab_sub_actuators.xacro (robot description, xacro)
@@ -42,29 +42,53 @@
      https://github.com/uuvsimulator/uuv_simulator/blob/5684de4827729f163f118cdc3a841011ef25ed8d/uuv_gazebo_plugins/uuv_gazebo_ros_plugins/src/ThrusterROSPlugin.cc#L153-L168 -->
 <!-- Top thrusters -->
-  <xacro:thruster_macro namespace="${namespace}" thruster_id="0"> <!-- heave back left prop up-->
+  <xacro:thruster_macro namespace="${namespace}" thruster_id="0">
   <origin xyz="-0.12070 0.12070 0" rpy="0 -1.5707963268 0"/>
   </xacro:thruster_macro>
-  <xacro:thruster_macro namespace="${namespace}" thruster_id="1"> <!-- heave bacl right prop up-->
+  <xacro:thruster_macro namespace="${namespace}" thruster_id="1">
     <origin xyz="-0.12070 -0.12070 0" rpy="0 -1.5707963268 0"/>
   </xacro:thruster_macro>
-  <xacro:thruster_macro namespace="${namespace}" thruster_id="2"> <!-- heave front left prop up-->
+  <xacro:thruster_macro namespace="${namespace}" thruster_id="2">
     <origin xyz="0.12070 0.12070 0" rpy="0 -1.5707963268 0"/>
   </xacro:thruster_macro>
-  <xacro:thruster_macro namespace="${namespace}" thruster_id="3"> <!-- heave front right prop up-->
+  <xacro:thruster_macro namespace="${namespace}" thruster_id="3">
     <origin xyz="0.12070 -0.12070 0" rpy="0 -1.5707963268 0"/>
   </xacro:thruster_macro>
+  <!-- <xacro:thruster_macro namespace="${namespace}" thruster_id="0">
+  <origin xyz="-0.143825 0.280455 0.230245" rpy="0 -1.5707963268 0"/>
+  </xacro:thruster_macro>
+  <xacro:thruster_macro namespace="${namespace}" thruster_id="1">
+    <origin xyz="-0.143825 -0.280455 0.230245" rpy="0 -1.5707963268 0"/>
+  </xacro:thruster_macro>
+  <xacro:thruster_macro namespace="${namespace}" thruster_id="2">
+    <origin xyz="0.143825 0.280455 0.230245" rpy="0 -1.5707963268 0"/>
+  </xacro:thruster_macro>
+  <xacro:thruster_macro namespace="${namespace}" thruster_id="3">
+    <origin xyz="0.143825 -0.280455 0.230245" rpy="0 -1.5707963268 0"/>
+  </xacro:thruster_macro> -->
  <!-- Front thrusters -->
-  <xacro:thruster_macro namespace="${namespace}" thruster_id="6"> <!-- lat front left-->
+  <xacro:thruster_macro namespace="${namespace}" thruster_id="6">
     <origin xyz="0.20506 0.20506 0" rpy="${0*d2r} ${0*d2r} ${135*d2r}"/>
   </xacro:thruster_macro>
-  <xacro:thruster_macro namespace="${namespace}" thruster_id="7"> <!-- lat front right -->
+  <xacro:thruster_macro namespace="${namespace}" thruster_id="7">
     <origin xyz="0.20506 -0.20506 0" rpy="${0*d2r} ${0*d2r} ${-135*d2r}"/>
   </xacro:thruster_macro>
+  <!-- <xacro:thruster_macro namespace="${namespace}" thruster_id="6">
+    <origin xyz="0.192247 0.286933 0.0721539" rpy="${0*d2r} ${0*d2r} ${135*d2r}"/>
+  </xacro:thruster_macro>
+  <xacro:thruster_macro namespace="${namespace}" thruster_id="7">
+    <origin xyz="0.192247 -0.286933 0.0721539" rpy="${0*d2r} ${0*d2r} ${-135*d2r}"/>
+  </xacro:thruster_macro> -->
  <!-- Back thrusters -->
-  <xacro:thruster_macro namespace="${namespace}" thruster_id="4"> <!-- lat back left-->
-    <origin xyz="-0.20506 0.20506 0" rpy="${0*d2r} ${0*d2r} ${45*d2r}"/>
+ <xacro:thruster_macro namespace="${namespace}" thruster_id="4"> <!-- lat back left-->
+   <origin xyz="-0.20506 0.20506 0" rpy="${0*d2r} ${0*d2r} ${45*d2r}"/>
+ </xacro:thruster_macro>
+ <xacro:thruster_macro namespace="${namespace}" thruster_id="5"> <!-- lat back right -->
+   <origin xyz="-0.20506 -0.20506 0" rpy="${0*d2r} ${0*d2r} ${-45*d2r}"/>
+ </xacro:thruster_macro>
+  <!-- <xacro:thruster_macro namespace="${namespace}" thruster_id="4">
+    <origin xyz="-0.192247 0.286933 0.0721539" rpy="${0*d2r} ${0*d2r} ${45*d2r}"/>
   </xacro:thruster_macro>
-  <xacro:thruster_macro namespace="${namespace}" thruster_id="5"> <!-- lat back right -->
-    <origin xyz="-0.20506 -0.20506 0" rpy="${0*d2r} ${0*d2r} ${-45*d2r}"/>
-  </xacro:thruster_macro>
+  <xacro:thruster_macro namespace="${namespace}" thruster_id="5">
+    <origin xyz="-0.192247 -0.286933 0.0721539" rpy="${0*d2r} ${0*d2r} ${-45*d2r}"/>
+  </xacro:thruster_macro> -->
 </robot>
